File: EMUPU_RAM68k/EMUPU_RAM68k.kicad_sch (KiCad schematic)
At the start: 22 parts, among them J3 Barrel_Jack_Switch, J4 Conn_01x06_Pin, J5 Conn_01x08_Pin, SW1 SW_SPDT, SW2 SW_SPST, U1 PIC18F47Q43-IP, U2 628128, U3 68008D_AA

Commit message: ram40_68k8 for B-board Rev. 002, just rebulided.
Parts:
- added R2: 10k, Resistor_THT:R_Axial_DIN0204_L3.6mm_D1.6mm_P7.62mm_Horizontal, symbol Device:R
- added TP1: TEST, TestPoint:TestPoint_THTPad_1.5x1.5mm_Drill0.7mm, symbol Connector:TestPoint_Small
- U3: footprint (none) -> 0-local:DIP-48_W15.24mm_Socket_OvalPad_splitcouryard
Connections:
- net BR: now also R2.2; no longer U1.28 (RD5)
- net GND: now also U2.22 (~{CS1})
- net VCC: now also R2.1; no longer U2.22 (~{CS1})
- new net TEST: TP1.1, U1.28 (RD5)
- no-connect marks 14 -> 15
Other:
- title: (none) -> 68008 on EMUPU_RAM40
Changed lines of the file:
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@@
 (kicad_sch (version 20230121) (generator eeschema)
   (paper "A4")
+  (title_block
+    (title "68008 on EMUPU_RAM40")
+    (date "2023-03-04")
+    (rev "002")
+  )
   (junction (at 223.52 87.63) (diameter 0) (color 0 0 0 0)
   )
@@
   (junction (at 102.87 53.34) (diameter 0) (color 0 0 0 0)
   )
-  (junction (at 152.4 119.38) (diameter 0) (color 0 0 0 0)
-  )
   (junction (at 102.87 78.74) (diameter 0) (color 0 0 0 0)
   )
@@
   )
   (junction (at 223.52 85.09) (diameter 0) (color 0 0 0 0)
+  )
+  (junction (at 88.9 134.62) (diameter 0) (color 0 0 0 0)
   )
   (junction (at 107.95 48.26) (diameter 0) (color 0 0 0 0)
@@
   (no_connect (at 86.36 45.72))
   (no_connect (at 40.64 71.12))
+  (no_connect (at 134.62 134.62))
   (no_connect (at 40.64 81.28))
   (wire (pts (xy 259.08 144.78) (xy 259.08 140.97))
@@
     (stroke (width 0) (type default))
   )
-  (wire (pts (xy 180.34 55.88) (xy 162.56 55.88))
-    (stroke (width 0) (type default))
-  )
   (wire (pts (xy 165.1 53.34) (xy 165.1 139.7))
     (stroke (width 0) (type default))
@@
     (stroke (width 0) (type default))
   )
-  (wire (pts (xy 86.36 134.62) (xy 162.56 134.62))
+  (wire (pts (xy 86.36 134.62) (xy 88.9 134.62))
     (stroke (width 0) (type default))
   )
@@
     (stroke (width 0) (type default))
   )
-  (wire (pts (xy 162.56 55.88) (xy 162.56 134.62))
-    (stroke (width 0) (type default))
-  )
   (wire (pts (xy 223.52 82.55) (xy 223.52 85.09))
     (stroke (width 0) (type default))
@@
     (stroke (width 0) (type default))
   )
-  (wire (pts (xy 147.32 119.38) (xy 152.4 119.38))
-    (stroke (width 0) (type default))
-  )
   (wire (pts (xy 86.36 48.26) (xy 107.95 48.26))
     (stroke (width 0) (type default))
@@
     (stroke (width 0) (type default))
   )
+  (wire (pts (xy 88.9 134.62) (xy 134.62 134.62))
+    (stroke (width 0) (type default))
+  )
+  (wire (pts (xy 156.21 119.38) (xy 156.21 120.65))
+    (stroke (width 0) (type default))
+  )
   (wire (pts (xy 266.7 144.78) (xy 259.08 144.78))
     (stroke (width 0) (type default))
@@
     (stroke (width 0) (type default))
   )
+  (wire (pts (xy 147.32 119.38) (xy 156.21 119.38))
+    (stroke (width 0) (type default))
+  )
   (wire (pts (xy 267.97 73.66) (xy 267.97 76.2))
     (stroke (width 0) (type default))
@@
   )
   (wire (pts (xy 147.32 53.34) (xy 153.67 53.34))
+    (stroke (width 0) (type default))
+  )
+  (wire (pts (xy 160.02 55.88) (xy 180.34 55.88))
     (stroke (width 0) (type default))
   )
@@
     (effects (font (size 1.27 1.27)) (justify left bottom))
   )
-  (label "BR" (at 173.99 55.88 0) (fields_autoplaced)
+  (label "TEST" (at 173.99 55.88 0) (fields_autoplaced)
     (effects (font (size 1.27 1.27)) (justify left bottom))
   )
@@
   (label "D0" (at 96.52 114.3 0) (fields_autoplaced)
     (effects (font (size 1.27 1.27)) (justify left bottom))
+  )
+  (symbol (lib_id "Device:R") (at 88.9 130.81 0) (unit 1)
+    (in_bom yes) (on_board yes) (dnp no) (fields_autoplaced)
+    (property "Reference" "R2" (at 90.678 130.1663 0)
+      (effects (font (size 1.27 1.27)) (justify left))
+    )
+    (property "Value" "10k" (at 90.678 132.0873 0)
+      (effects (font (size 1.27 1.27)) (justify left))
+    )
+    (property "Footprint" "Resistor_THT:R_Axial_DIN0204_L3.6mm_D1.6mm_P7.62mm_Horizontal" (at 87.122 130.81 90)
+      (effects (font (size 1.27 1.27)) hide)
+    )
+    (property "Datasheet" "~" (at 88.9 130.81 0)
+      (effects (font (size 1.27 1.27)) hide)
+    )
+    (pin "1")
+    (pin "2")
+    (instances
+      (project "EMUPU_RAM"
+        (path "/6d2188b2-a6ec-4341-9e2f-19ddbe5554d2"
+          (reference "R2") (unit 1)
+        )
+      )
+      (project "EMUPU_RAM68k"
+        (path "/e6d6b00c-3eac-46b2-864a-d30920c7bbcf"
+          (reference "R8") (unit 1)
+        )
+      )
+    )
   )
   (symbol (lib_id "Connector:Barrel_Jack_Switch") (at 269.24 30.48 0) (mirror y) (unit 1)
@@
     )
   )
+  (symbol (lib_id "power:VCC") (at 88.9 127 0) (unit 1)
+    (in_bom yes) (on_board yes) (dnp no) (fields_autoplaced)
+    (property "Reference" "#PWR012" (at 88.9 130.81 0)
+      (effects (font (size 1.27 1.27)) hide)
+    )
+    (property "Value" "VCC" (at 88.9 123.4981 0)
+      (effects (font (size 1.27 1.27)))
+    )
+    (property "Footprint" "" (at 88.9 127 0)
+      (effects (font (size 1.27 1.27)) hide)
+    )
+    (property "Datasheet" "" (at 88.9 127 0)
+      (effects (font (size 1.27 1.27)) hide)
+    )
+    (pin "1")
+    (instances
+      (project "EMUPU_RAM"
+        (path "/6d2188b2-a6ec-4341-9e2f-19ddbe5554d2"
+          (reference "#PWR012") (unit 1)
+        )
+      )
+      (project "EMUPU_RAM68k"
+        (path "/e6d6b00c-3eac-46b2-864a-d30920c7bbcf"
+          (reference "#PWR025") (unit 1)
+        )
+      )
+    )
+  )
   (symbol (lib_id "power:GND") (at 250.19 144.78 0) (unit 1)
     (in_bom yes) (on_board yes) (dnp no) (fields_autoplaced)
@@
     )
   )
+  (symbol (lib_id "Connector:TestPoint_Small") (at 160.02 55.88 0) (unit 1)
+    (in_bom yes) (on_board yes) (dnp no) (fields_autoplaced)
+    (property "Reference" "TP1" (at 161.163 55.2363 0)
+      (effects (font (size 1.27 1.27)) (justify left))
+    )
+    (property "Value" "TEST" (at 161.163 57.1573 0)
+      (effects (font (size 1.27 1.27)) (justify left))
+    )
+    (property "Footprint" "TestPoint:TestPoint_THTPad_1.5x1.5mm_Drill0.7mm" (at 165.1 55.88 0)
+      (effects (font (size 1.27 1.27)) hide)
+    )
+    (property "Datasheet" "~" (at 165.1 55.88 0)
+      (effects (font (size 1.27 1.27)) hide)
+    )
+    (pin "1")
+    (instances
+      (project "EMUPU_RAM68k"
+        (path "/e6d6b00c-3eac-46b2-864a-d30920c7bbcf"
+          (reference "TP1") (unit 1)
+        )
+      )
+    )
+  )
   (symbol (lib_id "0-local:68008D_AA") (at 63.5 101.6 0) (unit 1)
     (in_bom yes) (on_board yes) (dnp no) (fields_autoplaced)
@@
       (effects (font (size 1.27 1.27)))
     )
-    (property "Footprint" "" (at 63.5 78.74 0)
+    (property "Footprint" "0-local:DIP-48_W15.24mm_Socket_OvalPad_splitcouryard" (at 63.5 78.74 0)
       (effects (font (size 1.27 1.27)) hide)
     )
@@
         )
       )
+    )
+  )
+  (symbol (lib_id "power:GND") (at 156.21 120.65 0) (unit 1)
+    (in_bom yes) (on_board yes) (dnp no) (fields_autoplaced)
+    (property "Reference" "#PWR01" (at 156.21 127 0)
+      (effects (font (size 1.27 1.27)) hide)
+    )
+    (property "Value" "GND" (at 156.21 124.7855 0)
+      (effects (font (size 1.27 1.27)))
+    )
+    (property "Footprint" "" (at 156.21 120.65 0)
+      (effects (font (size 1.27 1.27)) hide)
+    )
+    (property "Datasheet" "" (at 156.21 120.65 0)
+      (effects (font (size 1.27 1.27)) hide)
+    )
+    (pin "1")
+    (instances
+      (project "EMUPU_RAM"
+        (path "/6d2188b2-a6ec-4341-9e2f-19ddbe5554d2"
+          (reference "#PWR01") (unit 1)
+        )
+      )
+      (project "EMUPU_RAM68k"
+        (path "/e6d6b00c-3eac-46b2-864a-d30920c7bbcf"
+          (reference "#PWR024") (unit 1)
+        )
+      )
