File: EMUPU_RAM.kicad_pcb (KiCad board)
At the start: 2 copper layers, 99.1 x 82.5 mm, 30 parts, among them J1 Conn_01x20_Socket, J2 Conn_01x20_Socket, J3 Barrel_Jack_Switch, J4 Conn_01x06_Pin, J5 Conn_01x08_Pin, J6 Conn_01x06_Pin, J7 Conn_01x02_Pin, SW1 SW_SPDT, SW2 SW_SPST, U2 HM678127_SOJ32_Arranged, U3 PIC18F57Q43-IPT

Commit message: RAM48-Rev003: direct ready for production
Parts:
- removed REF**: DIP-48_W15.24mm_Socket_OvalPad_nocourtyard, 0-local:DIP-48_W15.24mm_Socket_OvalPad_splitcouryard
- added D3: HALT, LED_THT:LED_D3.0mm, F.Cu at (105.4, 87.6)
- added D4: RESET, LED_THT:LED_D3.0mm, F.Cu at (105.4, 82.5)
- added D5: BUSAK, LED_THT:LED_D3.0mm, F.Cu at (105.4, 77.5)
- added JP1: SolderJumper_2_Bridged, Jumper:SolderJumper-2_P1.3mm_Bridged_RoundedPad1.0x1.5mm, F.Cu at (178.4, 132.1)
- added JP2: SolderJumper_2_Bridged, Jumper:SolderJumper-2_P1.3mm_Bridged_RoundedPad1.0x1.5mm, F.Cu at (178.4, 129.5)
- added JP3: SolderJumper_2_Bridged, Jumper:SolderJumper-2_P1.3mm_Bridged_RoundedPad1.0x1.5mm, F.Cu at (136.5, 132.1)
- added R10: 10k, Resistor_THT:R_Axial_DIN0204_L3.6mm_D1.6mm_P7.62mm_Horizontal, F.Cu at (101.5, 131.6)
- added R11: 10k, Resistor_THT:R_Axial_DIN0204_L3.6mm_D1.6mm_P7.62mm_Horizontal, F.Cu at (114.4, 131.6)
- added R7: 1.5k, Resistor_THT:R_Axial_DIN0204_L3.6mm_D1.6mm_P7.62mm_Horizontal, F.Cu at (123.2, 83.8)
- added R8: 1.5k, Resistor_THT:R_Axial_DIN0204_L3.6mm_D1.6mm_P7.62mm_Horizontal, F.Cu at (120.7, 83.8)
- added R9: 1.5k, Resistor_THT:R_Axial_DIN0204_L3.6mm_D1.6mm_P7.62mm_Horizontal, F.Cu at (118.1, 83.8)
- added U4: DIP-48_W15.24mm_Socket_OvalPad_nocourtyard, 0-Project:DIP-48_W15.24mm_Socket_OvalPad_splitcouryard, F.Cu at (152.4, 73.7)
- J3: footprint 0-local:BARREL_JACK -> 0-Project:BARREL_JACK
- J4, J6: footprint 0-local:PinHeader_1x06_P2.54mm_Horizontal_NoFeet -> 0-Project:PinHeader_1x06_P2.54mm_Horizontal_NoFeet
- J5: footprint 0-local:PinHeader_1x08_P2.54mm_Rev_Horizontal_Nofoot -> 0-Project:PinHeader_1x08_P2.54mm_Rev_Horizontal_Nofoot
- SW1: footprint 0-local:PowerSW_for_SBC_series -> 0-Project:PowerSW_for_SBC_series
- SW2: footprint 0-local:SW_PUSH_6mm_H4.3mm -> 0-Project:SW_PUSH_6mm_H4.3mm
- U3: footprint 0-local:Quad-2x6 -> 0-Project:Quad-2x6
- moved SW2 22.5 mm to (126.7, 60.9), turned to -90 degrees
- moved D2 10.6 mm to (116.2, 67.3)
- moved SW1 8.54 mm to (115.6, 61.6), turned to 0 degrees
- moved C3 5.24 mm to (96.5, 73.7), turned to -90 degrees
- moved J4 5.08 mm to (96.5, 69.8)
- moved D1 1.27 mm to (130.8, 73.7)
- moved J5 1.27 mm to (130.7, 69.9)
- moved J6 1.27 mm to (158.8, 69.8)
- moved R2 1.27 mm to (138.4, 73.7)
- moved R3 1.27 mm to (141.0, 73.7)
- moved R5 1.27 mm to (146.1, 73.7)
- moved R1 1.27 mm to (135.9, 73.7)
- moved R4 1.27 mm to (143.5, 81.3)
- moved R6 0.51 mm to (111.8, 131.6)
Connections:
- J5 pad 5: /TEST -> /~{INT}
- R5 pad 2: Net-(U2-~{OE}) -> Net-(JP1-B)
- U2 pad 28: Net-(U2-~{OE}) -> Net-(JP1-B)
- U2 pad 5: GND -> Net-(JP3-A)
- U3 pad 16: /~{RFSH} -> unconnected-(U3-RB4-Pad16)
- U3 pad 17: /~{M1} -> /~{RFSH}
- U3 pad 18: /TEST -> /~{INT}
- U3 pad 25: Net-(U2-~{OE}) -> /~{M1}
- U3 pad 26: /~{RD} -> Net-(JP1-B)
- U3 pad 29: /~{INT} -> /TEST
Routing:
- net Net-(JP1-B): track 0.00 -> 162.8 mm, vias 0 -> 6
- net /~{BUSAK}: track 0.00 -> 135.4 mm, vias 0 -> 2
- net /~{HALT}: track 0.00 -> 87.7 mm, vias 0 -> 4
- net /~{RD}: track 85.9 -> 8.05 mm, vias 4 -> 1
- net Net-(U2-~{OE}): track 72.8 -> 0.00 mm, vias 3 -> 0
- net Net-(JP2-B): track 56.4 -> 128.4 mm, vias 1 -> 3
- net /~{INT}: track 50.1 -> 113.2 mm
- net /~{RESET}: track 68.4 -> 111.7 mm, vias 2 -> 4
- net Net-(JP3-A): track 0.00 -> 41.8 mm, vias 0 -> 2
- net /A15: track 129.7 -> 88.6 mm
- net GND: track 399.6 -> 359.3 mm, vias 8 -> 7
- net Net-(J5-Pin_1): track 98.9 -> 130.7 mm, vias 7 -> 6
- net /TEST: track 133.2 -> 158.6 mm, vias 3 -> 5
- net Net-(D3-A): track 0.00 -> 25.1 mm
- net /~{MREQ}: track 58.2 -> 82.5 mm, vias 2 -> 4
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Other:
- board text added: "BUSAK"
- board text added: "HALT"
- board text added: "RESET"
- board text added: "Rev. 003 (DIRECT)"
- board text removed: "1.5k"
- board text removed: "10k"
- board text removed: "Rev. 002"
