File: EMUPU_RAM.kicad_sch (KiCad schematic)
At the start: 25 parts, among them J1 Conn_01x20_Socket, J2 Conn_01x20_Socket, J3 Barrel_Jack_Switch, J4 Conn_01x06_Pin, J5 Conn_01x08_Pin, J6 Conn_01x06_Pin, J7 Conn_01x02_Pin, SW1 SW_SPDT, SW2 SW_SPST, U2 HM678127_SOJ32_Arranged, U3 PIC18F57Q43-IPT

Commit message: RAM48-Rev003: direct ready for production
Parts:
- added D3: HALT, LED_THT:LED_D3.0mm, symbol Device:LED
- added D4: RESET, LED_THT:LED_D3.0mm, symbol Device:LED
- added D5: BUSAK, LED_THT:LED_D3.0mm, symbol Device:LED
- added JP1, JP2, JP3: SolderJumper_2_Bridged, Jumper:SolderJumper-2_P1.3mm_Bridged_RoundedPad1.0x1.5mm, symbol Jumper:SolderJumper_2_Bridged
- added R10, R11: 10k, Resistor_THT:R_Axial_DIN0204_L3.6mm_D1.6mm_P7.62mm_Horizontal, symbol Device:R
- added R7, R8, R9: 1.5k, Resistor_THT:R_Axial_DIN0204_L3.6mm_D1.6mm_P7.62mm_Horizontal, symbol Device:R
- J3: footprint 0-local:BARREL_JACK -> 0-Project:BARREL_JACK
- J4, J6: footprint 0-local:PinHeader_1x06_P2.54mm_Horizontal_NoFeet -> 0-Project:PinHeader_1x06_P2.54mm_Horizontal_NoFeet
- J5: footprint 0-local:PinHeader_1x08_P2.54mm_Rev_Horizontal_Nofoot -> 0-Project:PinHeader_1x08_P2.54mm_Rev_Horizontal_Nofoot
- SW1: footprint 0-local:PowerSW_for_SBC_series -> 0-Project:PowerSW_for_SBC_series
- SW2: footprint 0-local:SW_PUSH_6mm_H4.3mm -> 0-Project:SW_PUSH_6mm_H4.3mm
- U3: footprint 0-local:Quad-2x6 -> 0-Project:Quad-2x6
Connections:
- net GND: no longer U2.5 (~{CS})
- net TEST: now also U3.29 (RE2); no longer J5.5 (Pin_5), U3.18 (RB6/ICSPCLK)
- net VCC: now also R10.1, R11.1, R7.1, R8.1, R9.1
- net ~{BUSAK}: now also D5.1 (K)
- net ~{HALT}: now also D3.1 (K)
- net ~{INT}: now also J5.5 (Pin_5), U3.18 (RB6/ICSPCLK); no longer U3.29 (RE2)
- net ~{IORQ}: now also R11.2
- net ~{M1}: now also U3.25 (RA4); no longer U3.17 (RB5)
- net ~{MREQ}: now also JP3.2 (B), R10.2
- net ~{RD}: now also JP1.1 (A); no longer U3.26 (RA5)
- net ~{RESET}: now also D4.1 (K)
- net ~{RFSH}: now also U3.17 (RB5); no longer U3.16 (RB4)
- net ~{WR}: now also JP2.1 (A)
- net at R5.2, U2.28 (~{OE}): now also U3.26 (RA5), JP1.2 (B); no longer U3.25 (RA4)
- net at R6.2, U2.12 (~{WE}), U3.23 (RA2): now also JP2.2 (B)
- new net: D4.2 (A), R8.2
- new net: D3.2 (A), R7.2
- new net: D5.2 (A), R9.2
- new net: JP3.1 (A), U2.5 (~{CS})
- no-connect marks 11 -> 9
Other:
- note added: "CLK"
- note added: "TEST"
- note added: "~{BUSRQ}"
- note added: "~{IORQ}"
- note added: "~{M1}"
- note added: "~{MREQ}"
- note added: "~{RD}"
- note added: "~{RESET}"
- note added: "~{WR}"
- title: EMUPU_RAM48 board -> EMUPU_RAM48 board (DIRECT)
- moved on the sheet: C4, C5, R5, R6
